File: KiCAD/espRGB/espRGB.sch (KiCad schematic (older format))
At the start: 16 parts, among them J1 Conn_01x04_Female, J2 Conn_01x02_Female, Q1 Q_PNP_BEC, Q2 Q_NPN_BEC, Q3 Q_PNP_BEC, Q4 Q_NPN_BEC, Q5 Q_PNP_BEC, Q6 Q_NPN_BEC, Q7 Q_NMOS_GSD, Q8 Q_NMOS_GSD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

Commit message: v1.1
Parts:
- removed J1: Conn_01x04_Female, TerminalBlock_Phoenix:TerminalBlock_Phoenix_MKDS-1,5-4-5.08_1x04_P5.08mm_Horizontal, symbol Connector:Conn_01x04_Female
- removed J2: Conn_01x02_Female, TerminalBlock_Phoenix:TerminalBlock_Phoenix_MKDS-1,5-2-5.08_1x02_P5.08mm_Horizontal, symbol Connector:Conn_01x02_Female
- removed Q1, Q3, Q5: Q_PNP_BEC, Package_TO_SOT_SMD:SOT-23, symbol Device:Q_PNP_BEC
- removed Q2, Q4, Q6: Q_NPN_BEC, Package_TO_SOT_SMD:SOT-23, symbol Device:Q_NPN_BEC
- removed Q7, Q8, Q9: Q_NMOS_GSD, Package_TO_SOT_SMD:SOT-223-3_TabPin2, symbol Device:Q_NMOS_GSD
- removed R1, R2, R3: R, Resistor_SMD:R_0603_1608Metric, symbol Device:R
- added J? (x2): Conn_01x04_Female, symbol Connector:Conn_01x04_Female
- added J? (x3): Conn_01x02_Female, symbol Connector:Conn_01x02_Female
- added Q? (x6): Q_NMOS_GDS, symbol Device:Q_NMOS_GDS
- added R? (x2): R, symbol Device:R
Connections:
- net +12V: now also J?.1 (Pin_1), J?.1 (Pin_1), J?.1 (Pin_1)
- net GND: now also J?.2 (Pin_2), J?.2 (Pin_2), J?.2 (Pin_2), Q?.3 (S), Q?.3 (S), Q?.3 (S), Q?.3 (S), Q?.3 (S), Q?.3 (S)
- net red2_gate: now reaches U1.13 (SDA/D2)
- net red2_gate: now also Q?.1 (G)
- net blue2_gate: now reaches U1.14 (SCL/D1)
- net blue2_gate: now also Q?.1 (G)
- net blue1_gate: now reaches U1.4 (SCK/D5)
- net blue1_gate: now also Q?.1 (G)
- net red1_gate: now reaches U1.5 (MISO/D6)
- net red1_gate: now also Q?.1 (G)
- net green1_gate: now reaches U1.6 (MOSI/D7)
- net green1_gate: now also Q?.1 (G)
- net button1: now reaches U1.7 (CS/D8)
- net button1: now also J?.1 (Pin_1), R?.2
- net +3V3: now reaches U1.8 (3V3)
- net +3V3: now also R?.1, R?.1
- net blue: no longer names the net of U1.3 (D0)
- net green renamed button2
- net button2: now also J?.1 (Pin_1), R?.2
- net red renamed green2_gate
- net green2_gate: now also Q?.1 (G)
- new net blue1: J?.4 (Pin_4), Q?.2 (D)
- new net blue2: J?.4 (Pin_4), Q?.2 (D)
- new net green1: J?.2 (Pin_2), Q?.2 (D)
- new net green2: J?.2 (Pin_2), Q?.2 (D)
- new net red1: J?.3 (Pin_3), Q?.2 (D)
- new net red2: J?.3 (Pin_3), Q?.2 (D)
- no-connect marks 4 -> 3
Other:
- note removed: "Terminal block"
- moved on the sheet: U1, VR1
